File: PCB_KioskMB_r3.2.brd (EAGLE design)
At the start: 146.1 x 101.9 mm, 340 parts, among them IC1 ISL60002DIH325Z-TK, IC18 FT232RL, IC19 MCP6022-I/ST, IC2 SN65HVD12D, IC20 LTC1771EMS8, IC21 LTC1771EMS8, IC3 PIC24FJ256GA110-I/PT, IC4 PIC10F200T-I/OT, IC5 LM75ADP, IC6 24LC32A-I/MS, IC7 PCF2123TS/1-T, IC8 M25P16-VMN6P, IC9 LM3405AXMK/NOPB, J1 DF11-10DP-2DSA(01), J10 CCM03-3504LFT-NR, J13 3-641215-3, J14 3-641215-2, J15 3-641215-4, J16 3-641215-4, J40 DNP, J43 3-641215-4, J44 3-641215-4, J45 3-641215-4, J46 3-641215-5, J47 DF11-10DP-2DSA(01), J48 3-641215-2, J49 3-641215-2, J5 3-641215-2, J6 3-641215-2, J7 SS-6566-NF, J8 TSW-108-07-G-D, J9 SS-6566-NF, Q1 SSM6P49NU,LFPZ, Q14 TSM9938HEUK+T, Q15 SI4564DY, Q16 CSD87331Q3D, Q17 TSM9938HEUK+T, Q18 SI4564DY, Q19 CSD87331Q3D, Q2 FDC6330L, Q20 IPD30N06S2L-23, Q21 IPD30N06S2L-23, Q22 FDN352AP, Q23 FDN352AP, Q24 BSS138, Q3 SR3.3.TCT, Q4 7B-28.63636MAAJ-T, Q5 FDC6324L, Q6 CM519 32.768KDZF-UT, Q7 SSM6P49NU,LFPZ, Q8 IPD30N06S2L-23, Q9 IPD30N06S2L-23, U1 LTC1955, U2 HRXL-MAXSONAR-WRC-MB7387, U3 ADS1015, U6 TPS43061, U7 TPS43061, U8 TPA3111D1PWP, U9 OPA322SAIDBVT, X1 FH12-10S-0.5S1.00MM

Commit message: save state 12:27pm
save state 12:27pm
Routing:
- net SDA1: track 29.6 -> 121.8 mm, vias 0 -> 5
- net U1RX: track 20.7 -> 108.3 mm, vias 0 -> 4
- net DCDC_12V_EN: track 32.5 -> 118.6 mm, vias 2 -> 3
- net U1TX: track 14.6 -> 97.1 mm, vias 0 -> 4
- net MH_STROBE: track 10.5 -> 92.9 mm, vias 0 -> 1
- net SCL1: track 39.2 -> 120.5 mm, vias 0 -> 5
- net MH_DATA: track 10.9 -> 90.5 mm, vias 0 -> 1
- net +SMB: track 197.8 -> 237.9 mm
- net US-S_O: track 0.00 -> 22.6 mm
- net N$72: track 5.10 -> 21.5 mm, vias 0 -> 2
- net DOOR_ON: track 6.75 -> 17.7 mm
- net U2CTL: track 106.3 -> 107.9 mm
- net U2TX: track 56.6 -> 58.1 mm
- net U2RX: track 47.9 -> 49.3 mm

Commit message: update from thursday
update from thursday
Parts:
- moved R167 0.46 mm to (52.5, 50.0)
Routing:
- net +3.3V: track 315.3 -> 451.7 mm, vias 17 -> 25
- net +3.3V/2: track 107.6 -> 200.9 mm, vias 5 -> 7
- net +SMB: track 237.9 -> 323.4 mm
- net 5V_ON: track 5.67 -> 84.9 mm, vias 0 -> 1
- net SDA1: track 121.8 -> 198.6 mm, vias 5 -> 6
- net SCL1: track 120.5 -> 191.0 mm, vias 5 -> 6
- net ID_PWM: track 8.16 -> 67.1 mm, vias 0 -> 2
- net DGND: track 310.3 -> 363.3 mm, vias 125 -> 138
- net B12_PG: track 15.3 -> 62.5 mm, vias 0 -> 2
- net +3.3V/1: track 233.3 -> 277.6 mm, vias 6 -> 8
- net VPS_ON: track 40.3 -> 81.5 mm, vias 2 -> 4
- net SCLK2: track 68.8 -> 99.7 mm
- net STR_PG: track 15.1 -> 43.1 mm, vias 0 -> 2
- net DCDC12VIN: track 16.8 -> 37.7 mm
- net N$63: track 4.05 -> 19.6 mm
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