File: PCB_KioskMB_r3.2.brd (EAGLE design)
At the start: 157 x 103 mm, 340 parts, among them CN2 0039301040, IC1 ISL60002DIH325Z-TK, IC18 FT232RL, IC19 MCP6022-I/ST, IC2 SN65HVD12D, IC20 LTC1771EMS8, IC21 LTC1771EMS8, IC3 PIC24FJ256GA110-I/PT, IC4 PIC10F200T-I/OT, IC5 LM75ADP, IC6 24LC32A-I/MS, IC7 PCF2123TS/1-T, IC8 M25P16-VMN6P, IC9 LM3405AXMK/NOPB, J1 DF11-10DP-2DSA(01), J10 CCM03-3504LFT-NR, J13 3-641215-3, J14 3-641215-2, J15 3-641215-4, J16 3-641215-4, J43 3-641215-4, J44 3-641215-4, J45 3-641215-4, J46 3-641215-5, J47 DF11-10DP-2DSA(01), J48 3-641215-2, J49 3-641215-2, J5 3-641215-2, J6 3-641215-2, J7 SS-6566-NF, J8 TSW-108-07-G-D, J9 SS-6566-NF, Q14 TSM9938HEUK+T, Q15 SI4564DY, Q16 CSD87331Q3D, Q17 TSM9938HEUK+T, Q18 SI4564DY, Q19 CSD87331Q3D, Q2 FDC6330L, Q20 IPD30N06S2L-23, Q21 IPD30N06S2L-23, Q22 FDN352AP, Q23 FDN352AP, Q24 BSS138, Q3 SR3.3.TCT, Q4 7B-28.63636MAAJ-T, Q5 FDC6324L, Q6 CM519 32.768KDZF-UT, Q7 SSM6P49NU,LFPZ, Q8 IPD30N06S2L-23, Q9 IPD30N06S2L-23, U1 LTC1955, U2 HRXL-MAXSONAR-WRC-MB7387, U3 ADS1015, U6 TPS43061, U7 TPS43061, U8 TPA3111D1PWP, U9 OPA322SAIDBVT, X1 FH12-10S-0.5S1.00MM, X2 MINI-USB_4P-85-32004-10X

Commit message: push latest
Parts:
- removed J50: (no value), CON-PhoenixContac-AON:TERM-2
- moved CN2 123.5 mm to (14.0, 50.0), turned to 270 degrees
- moved R36 10.5 mm to (24.3, 64.4)
- moved R31 10.4 mm to (19.2, 61.4)
- moved R32 10.4 mm to (20.6, 55.8)
- moved R33 10.4 mm to (27.3, 59.1)
- moved R34 10.4 mm to (25.2, 59.1)
- moved R35 10.4 mm to (25.6, 62.4)
- moved U3 10.4 mm to (22.3, 60.1)
- moved C37 10.3 mm to (20.3, 64.9)
Connections:
- net DGND: now also CN2.1, CN2.2; no longer J50.1
- net P12V: now also CN2.3, CN2.4; no longer J50.2
Routing:
- net +3.3V/1: track 275.1 -> 237.7 mm, vias 7 -> 6
- net SDA1: track 223.6 -> 203.6 mm, vias 10 -> 8
- net SCL1: track 205.2 -> 193.3 mm
- net BAT_SENSE: track 50.6 -> 62.2 mm
- net BAT_GND: track 61.2 -> 69.8 mm
- net P12V: track 170.0 -> 161.5 mm
- net +5V: track 75.2 -> 67.2 mm
- net 18V_SENSE: track 53.3 -> 50.0 mm, vias 2 -> 1
- net 18V_GND: track 63.0 -> 60.5 mm, vias 1 -> 0
- net N$21: track 5.57 -> 4.55 mm
- net DGND: track 402.4 -> 401.6 mm, vias 137 -> 136

Commit message: new rev number
major changes, reviewed all of Jarv's notes and applied them. started changing connectors.
Parts:
- removed C151: 1nF, discrete:0603
- removed C159: 5pF, discrete:0603
- removed C161: 0.1uF, discrete:0603
- removed C162: 220pF, discrete:0603
- removed C36: 10uF/35V, discrete:1206
- removed CN1: (no value), adafruit:DCJACK_2MM_PTH
- removed D29: STPS0540Z, st-microelectronics-AOM:SOD-123
- removed D5, D6: SS14, Vishay-AON:SMA
- removed D7, D8: LED-GR, discrete:0805-POL
- removed D9: SMAJ26A, DiodesInc-AON:SMA
- removed IC20: LTC1771EMS8, LinearTech-AON:MSOP-08
- removed J15, J16: 3-641215-4, Tyco-U:3-641215-4
- removed L13: CR75-330KC, Sumida-UT:CR75
- removed Q22: FDN352AP, Fairchild-AON:SOT-23
- removed Q8, Q9: IPD30N06S2L-23, InfineonTech-AON:TO252
- removed R153, R155, R169: CSR1206FK25L0, Brenneman:R1206
- removed R188: 0.12R, discrete:0805
- removed R191: 10K, discrete:0603
- removed R192: 1.65M, discrete:0603
- removed R196, R29, R30: 1M, discrete:0603
- removed R27, R28: 3.3K, discrete:0805
- removed TP68: TPB1,27, testpad:B1,27
- added C3, C38, C39, C41: 10uF/4V, discrete:0603
- added C40, C42: 0.1uF, discrete:0603
- added C43: 470uF/35-50V, resistor:E5-13
- added C44: 220uF, 16V, AL, resistor:153CLV-0605
- added C45: 10uF, discrete:1210
- added C46: 0.1uF, discrete:1210
- added H6: STANDOFF_ELECTRICAL, SparkFun-Hardware:STANDOFF-ELECTRICAL
- added J30: 22-11-2072, elocktech_lib:HRXL-MAXSONAR-WRC-MB7387
- added JP1: (no value), ChipTestJig:1X02_2.54_SCREWTERM
- added R38, R39: 1K, discrete:0603
- added R40, R41, R42, R43, R44: 0.025R, discrete:0805
- added R45, R46: 470R, discrete:0603
- added R47: 0R, discrete:0603
- added R48: DNP, discrete:0603
- C29: value 10uF/10V -> 10uF/4V
- C4: value 100nF -> 0.1uF
- C7: value 1u/10V -> 10uF/4V
- C9: value 0.1uF -> 10uF/4V
- Q14, Q17: value TSM9938HEUK+T -> MAX9938HEUK
- Q5: value FDC6324L -> FDC6330L
- R1: value 47R -> 300R
- R31, R32: value 1M -> 10K
- U2: value HRXL-MAXSONAR-WRC-MB7387 -> LE33; device elocktech_lib:HRXL-MAXSONAR-WRC-MB7387 -> elock_lib:LE33
- moved U2 78.2 mm to (39.1, 52.6), turned to 270 degrees
- moved R36 25.3 mm to (19.7, 39.5), turned to 270 degrees
- moved TP63 23.0 mm to (22.4, 12.7)
- moved R35 20.5 mm to (24.0, 41.9)
- moved C37 19.7 mm to (19.6, 45.2)
- moved R31 18.4 mm to (24.0, 43.6), turned to 0 degrees
- moved R34 18.4 mm to (15.2, 43.7), turned to 0 degrees
- moved R33 18.4 mm to (15.2, 45.3), turned to 180 degrees
- moved U3 17.7 mm to (19.6, 42.6), turned to 270 degrees
- moved C187 11.6 mm to (19.2, 23.7)
- moved CN2 11.4 mm to (14.0, 61.4)
- moved R32 11.2 mm to (24.0, 45.2), turned to 0 degrees
- moved TP64 9.86 mm to (33.4, 56.3)
- moved TP66 9.51 mm to (33.4, 48.9)
- moved FID1 3.86 mm to (1.86, 1.45)
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Connections:
- removed net GNDBREAK: CN1.GNDBREAK
- removed net N$12: D7.2, R27.1
- removed net N$15: D8.2, R28.1
- removed net N$27: IC20.5, Q22.1
- removed net N$29: IC20.2, R191.2
- removed net N$30: C162.1, R191.1
- removed net N$31: C161.1, IC20.1, TP68.TP
- removed net N$33: D29.C, L13.1, Q22.3
- removed net N$37: C151.2, IC20.7, Q22.2, R188.1
- removed net N$38: C159.1, IC20.3, R192.2, R196.1
- removed net N$53: Q17.5, Q18.5, Q18.6, R168.1
- removed net OUT_S3: D5.C, D7.1+, J15.2, J16.2, Q8.3
- removed net OUT_S4: D6.C, D8.1+, J15.3, J16.3, Q9.3
- new net N$41: JP1.P1, JP2.P1, R39.2
- new net N$42: J45.2, R46.2
- new net N$47: J45.3, R45.2
- new net N$48: C149.1, C150.1, C46.1, R47.1, R48.1, U2.8
- new net N$5: JP3.P1, JP4.P1, R38.2
- new net SMB-MEAS: Q17.4, Q18.3, R168.2, R170.1
- net +3.3V: now also C45.1, U2.1; no longer C159.2, L13.2, R192.1
- net +3.3V/2: now also J30.6; no longer U2.6
- net +5V: now also R47.2
- net +SMB: now also Q17.5, R168.1, R48.2; no longer C149.1, C150.1, C151.1, IC20.6, IC20.8, Q18.3, R170.1, R188.2
- net 18V_GND: now also C39.2, C40.1, R39.1; no longer CN1.GND, JP2.P1
- net 18V_SENSE: now also JP1.P2; no longer CN1.PWR
- net ACT_S3_B: no longer Q9.1, R30.1
- net ACT_S4_B: no longer Q8.1, R29.1
- net B12_FEED: now also R42.2, R43.2; no longer R153.2, R155.2
- net BAT_GND: now also C41.2, C42.1, R38.1; no longer JP3.P1, JP4.P1
- net DCDC12VIN: now also R40.2, R41.2, R42.1, R43.1; no longer R153.1, R155.1
- net DGND: now also C3.2, C38.1, C40.2, C42.2, C43.-, C44.-, C45.2, C46.2, J30.7, U2.2, U2.3, U2.5, U2.6; no longer C161.2, C162.2, C36.2, D25.A, D26.A, D29.A, D5.A, D6.A, D9.-, IC20.4, J15.1, J16.1, Q8.2, Q9.2, R196.2, R29.2, R30.2
- net N$1: now also C38.2
- net N$19: now also C39.1
- net N$21: now also C41.1
- net N$4: now also R40.1, R41.1
- net N$49: now also C3.1
- net N$9: now also J30.4; no longer U2.4
- net OUT_S1: now also D25.A; no longer D25.C
- net OUT_S2: now also D26.A; no longer D26.C
- net P12V: now also C44.+
- net SMB_SCL: now also R46.1; no longer J45.2
- net SMB_SDA: now also R45.1; no longer J45.3
- net STR_FEED: now also R44.2; no longer R169.2
- net US-S_O: now also J30.5; no longer U2.5
- net VACT: now also C43.+, D25.C, D26.C; no longer C36.1, D9.+, J15.4, J16.4, R27.2, R28.2
- net VSUPLYACT: now also Q18.5, Q18.6, R44.1; no longer Q17.4, R168.2, R169.1
Routing:
- net ACT_S4_B: track 97.3 -> 0.00 mm, vias 4 -> 0
- net ACT_S3_B: track 80.5 -> 0.00 mm, vias 4 -> 0
- net BAT_GND: track 69.8 -> 15.9 mm, vias 1 -> 2
- net 18V_GND: track 60.5 -> 7.62 mm
- net +3.3V/1: track 237.7 -> 284.7 mm, vias 6 -> 10
- net N$5: track 0.00 -> 45.5 mm
- net VACT: track 194.1 -> 150.8 mm, vias 2 -> 5
- net OUT_S3: track 39.0 -> 0.00 mm
- net STR_FEED: track 13.0 -> 50.1 mm, vias 0 -> 2
- net OUT_S4: track 36.8 -> 0.00 mm
- net N$41: track 0.00 -> 35.7 mm
- net +5V: track 67.2 -> 99.6 mm, vias 3 -> 4
- net DCDC12VIN: track 43.3 -> 75.0 mm, vias 0 -> 2
- net 18V_SENSE: track 50.0 -> 28.9 mm, vias 1 -> 0
- net +3.3V: track 420.5 -> 441.4 mm, vias 26 -> 29
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- added copper zone on layer 1, net +SMB
- added copper zone on layer 1, net +SMB_PRE
- added copper zone on layer 1, net P12V
