File: PCB_KioskMB_r3.2.sch (EAGLE design)
At the start: 338 parts, among them IC1 ISL60002DIH325Z-TK, IC18 FT232RL, IC19 MCP6022-I/ST, IC2 SN65HVD12D, IC20 LTC1771EMS8, IC21 LTC1771EMS8, IC3 PIC24FJ256GA110-I/PT, IC4 PIC10F200T-I/OT, IC5 LM75ADP, IC6 24LC32A-I/MS, IC7 PCF2123TS/1-T, IC8 M25P16-VMN6P, IC9 LM3405AXMK/NOPB, J1 DF11-10DP-2DSA(01), J10 CCM03-3504LFT-NR, J13 3-641215-3, J14 3-641215-2, J15 3-641215-4, J16 3-641215-4, J43 3-641215-4, J44 3-641215-4, J45 3-641215-4, J46 3-641215-5, J47 DF11-10DP-2DSA(01), J48 3-641215-2, J49 3-641215-2, J5 3-641215-2, J6 3-641215-2, J7 SS-6566-NF, J8 TSW-108-07-G-D, J9 SS-6566-NF, Q14 TSM9938HEUK+T, Q15 SI4564DY, Q16 CSD87331Q3D, Q17 TSM9938HEUK+T, Q18 SI4564DY, Q19 CSD87331Q3D, Q2 FDC6330L, Q20 IPD30N06S2L-23, Q21 IPD30N06S2L-23, Q22 FDN352AP, Q23 FDN352AP, Q24 BSS138, Q3 SR3.3.TCT, Q4 7B-28.63636MAAJ-T, Q5 FDC6324L, Q6 CM519 32.768KDZF-UT, Q7 SSM6P49NU,LFPZ, Q8 IPD30N06S2L-23, Q9 IPD30N06S2L-23, U1 LTC1955, U2 HRXL-MAXSONAR-WRC-MB7387, U3 ADS1015, U6 TPS43061, U7 TPS43061, U8 TPA3111D1PWP, U9 OPA322SAIDBVT, X1 FH12-10S-0.5S1.00MM, X2 MINI-USB_4P-85-32004-10X

Commit message: added molex connector
Parts:
- removed H6: STANDOFF_ELECTRICAL, SparkFun-Hardware:STANDOFF_ELECTRICAL
- added CN2: 0039301040, elock_lib:0039301040
- added H1: STANDOFF_ELECTRICAL, SparkFun-Hardware:STANDOFF_ELECTRICAL
- C1, C10, C114, C115, C12, C121, C13, C134, C14, C15, C150, C151, C154, C155, C159, C16, C160, C161, C162, C163, C164, C17, C172, C18, C19, C2, C20, C21, C22, C23, C24, C25, C26, C28, C29, C30, C31, C32, C33, C34, C35, C37, C4, C5, C59, C6, C7, C8, C9: device DISCRETE:C-0603 -> discrete:C-0603
- C11: device DISCRETE:C-0805 -> discrete:C-0805
- C135, C142, C36: device DISCRETE:C-1206 -> discrete:C-1206
- C149, C152, C153, C157, C158, C27: device DISCRETE:C-1210 -> discrete:C-1210
- C156: device DISCRETE:C-POL-3528 -> discrete:C-POL-3528
- C187: device DISCRETE:ELC-7,5 -> resistor:CPOL-USE7.5-18
- D17, D19, D23, D24, D7, D8: device DISCRETE:LED-0805 -> discrete:LED-0805
- L1, L17, L2: device DISCRETE:L-1206 -> discrete:L-1206
- R1, R10, R11, R14, R151, R152, R170, R173, R174, R18, R183, R184, R187, R19, R190, R191, R192, R193, R194, R195, R196, R197, R22, R24, R29, R3, R30, R31, R32, R33, R34, R35, R36, R37, R4, R5, R6, R7, R8, R9: device DISCRETE:R-0603 -> discrete:R-0603
- R12, R13, R15, R16, R17, R23, R25, R26: device DISCRETE:R-0603-0RTOP -> discrete:R-0603-0RTOP
- R154, R168, R175, R176, R188, R189, R27, R28: device DISCRETE:R-0805 -> discrete:R-0805
- TP1, TP2, TP3, TP4, TP5, TP7, TP8: device TESTPAD:ROUND_SMD1MM -> testpad:ROUND_SMD1MM
- TP11, TP60, TP9: device TESTPAD:ROUND_SMD0.7MM -> testpad:ROUND_SMD0.7MM
- TP12: device TESTPAD:TP_0812 -> testpad:TP_0812
- TP61, TP62, TP63, TP64, TP65, TP66, TP67, TP68: value TP0.8 -> TPB1,27; device TESTPAD:TP0.8 -> testpad:TPB1,27
- TP69: device TESTPAD:P1-13 -> testpad:P1-13
Connections:
- net +SMB: now also C187.+; no longer C187.PIN+
- net DGND: now also C187.-, H1.P$1; no longer C187.PIN-, H6.P$1
Other:
- note added: "C187 is 16mm Can, 1mm dia. leads, 7.5 mm pitch"
- note added: "replace j50 with 4 pin (2x2) molex, similar to PSU"

Commit message: push latest
Parts:
- removed J50: (no value), CON-PhoenixContac-AON:TERM-2
Connections:
- net DGND: now also CN2.1, CN2.2; no longer J50.1
- net P12V: now also CN2.3, CN2.4; no longer J50.2
Other:
- moved on the sheet: CN2
Changed lines of the file:
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@@
 <part name="U$342" library="SUPPLY" deviceset="+3.3V/1" device=""/>
 <part name="C187" library="resistor" library_urn="urn:adsk.eagle:library:348" deviceset="CPOL-US" device="E7.5-18" value="2mF/16V"/>
-<part name="J50" library="CON-PhoenixContac-AON" deviceset="TERM-2" device=""/>
 <part name="U$47" library="SUPPLY" deviceset="DGND" device=""/>
 <part name="D32" library="Littelfuse" deviceset="P6SMB*" device="" technology="16A"/>
@@
 <wire x1="40.64" y1="58.42" x2="40.64" y2="60.96" width="0.1524" layer="94"/>
 <wire x1="38.1" y1="78.74" x2="38.1" y2="76.2" width="0.1524" layer="94"/>
-<text x="396.24" y="292.1" size="1.778" layer="94">replace j50 with 4 pin (2x2) molex, similar to PSU</text>
+<text x="393.7" y="274.32" size="1.778" layer="94">replace j50 with 4 pin (2x2) molex, similar to PSU</text>
 </plain>
 <instances>
@@
 <attribute name="VALUE" x="38.735" y="56.8325" size="1.27" layer="96"/>
 </instance>
-<instance part="J50" gate="J" x="391.16" y="294.64" rot="MR0"/>
-<instance part="U$47" gate="G$1" x="386.08" y="289.56" smashed="yes"/>
+<instance part="U$47" gate="G$1" x="386.08" y="279.4" smashed="yes"/>
 <instance part="D32" gate="G$1" x="48.26" y="53.34" smashed="yes" rot="R90">
 <attribute name="NAME" x="47.3075" y="46.7995" size="1.778" layer="95" rot="R90"/>
@@
 </instance>
 <instance part="U$97" gate="G$1" x="447.04" y="241.3" smashed="yes"/>
-<instance part="CN2" gate="G$1" x="406.4" y="307.34" rot="MR180"/>
+<instance part="CN2" gate="G$1" x="393.7" y="289.56" rot="MR180"/>
 </instances>
 <busses>
@@
 <pinref part="D20" gate="G$1" pin="K"/>
 <pinref part="TP61" gate="G$1" pin="TP"/>
-<pinref part="J50" gate="J" pin="2"/>
 <wire x1="360.68" y1="294.64" x2="386.08" y2="294.64" width="0.1524" layer="91"/>
 <junction x="360.68" y="294.64"/>
+<pinref part="CN2" gate="G$1" pin="4"/>
+<pinref part="CN2" gate="G$1" pin="3"/>
+<wire x1="386.08" y1="294.64" x2="388.62" y2="294.64" width="0.1524" layer="91"/>
+<wire x1="388.62" y1="292.1" x2="386.08" y2="292.1" width="0.1524" layer="91"/>
+<wire x1="386.08" y1="292.1" x2="386.08" y2="294.64" width="0.1524" layer="91"/>
+<junction x="386.08" y="294.64"/>
 </segment>
 </net>
@@
 </segment>
 <segment>
-<pinref part="J50" gate="J" pin="1"/>
 <pinref part="U$47" gate="G$1" pin="DGND"/>
+<pinref part="CN2" gate="G$1" pin="2"/>
+<wire x1="388.62" y1="287.02" x2="386.08" y2="287.02" width="0.1524" layer="91"/>
+<wire x1="386.08" y1="287.02" x2="386.08" y2="284.48" width="0.1524" layer="91"/>
+<wire x1="386.08" y1="284.48" x2="386.08" y2="281.94" width="0.1524" layer="91"/>
+<pinref part="CN2" gate="G$1" pin="1"/>
+<wire x1="388.62" y1="284.48" x2="386.08" y2="284.48" width="0.1524" layer="91"/>
+<junction x="386.08" y="284.48"/>
 </segment>
 <segment>

Commit message: new rev number
major changes, reviewed all of Jarv's notes and applied them. started changing connectors.
Parts:
- removed C151: 1nF, discrete:C-0603
- removed C159: 5pF, discrete:C-0603
- removed C161: 0.1uF, discrete:C-0603
- removed C162: 220pF, discrete:C-0603
- removed C36: 10uF/35V, discrete:C-1206
- removed CN1: (no value), adafruit:DCBARRELPTH
- removed D29: STPS0540Z, st-microelectronics-AOM:STPS0540Z
- removed D5, D6: SS14, Vishay-AON:SS14
- removed D7, D8: LED-GR, discrete:LED-0805
- removed D9: SMAJ26A, DiodesInc-AON:SMAJ5.0A
- removed IC20: LTC1771EMS8, LinearTech-AON:LTC1771EMS8
- removed J15, J16: 3-641215-4, Tyco-U:3-641215-4
- removed L13: CR75-330KC, Sumida-UT:CR75-330KC
- removed Q22: FDN352AP, Fairchild-AON:FDN352AP
- removed Q8, Q9: IPD30N06S2L-23, InfineonTech-AON:IPD30N06S2L-23
- removed R153, R155, R169: CSR1206FK25L0, Brenneman:R-US_R1206
- removed R188: 0.12R, discrete:R-0805
- removed R191: 10K, discrete:R-0603
- removed R192: 1.65M, discrete:R-0603
- removed R196, R29, R30: 1M, discrete:R-0603
- removed R27, R28: 3.3K, discrete:R-0805
- removed TP68: TPB1,27, testpad:TPB1,27
- added C3, C38, C39, C41: 10uF/4V, discrete:C-0603
- added C40, C42: 0.1uF, discrete:C-0603
- added C43: 470uF/35-50V, resistor:CPOL-USE5-13
- added C44: 220uF, 16V, AL, resistor:CPOL-US153CLV-0605
- added C45: 10uF, discrete:C-1210
- added C46: 0.1uF, discrete:C-1210
- added H6: STANDOFF_ELECTRICAL, SparkFun-Hardware:STANDOFF_ELECTRICAL
- added J30: 22-11-2072, elocktech_lib:HRXL-MAXSONAR-WRC-MB7387
- added JP1: (no value), ChipTestJig:M022.54MM_SCREWTERM
- added R38, R39: 1K, discrete:R-0603
- added R40, R41, R42, R43, R44: 0.025R, discrete:R-0805
- added R45, R46: 470R, discrete:R-0603
- added R47: 0R, discrete:R-0603
- added R48: DNP, discrete:R-0603
- C29: value 10uF/10V -> 10uF/4V
- C4: value 100nF -> 0.1uF
- C7: value 1u/10V -> 10uF/4V
- C9: value 0.1uF -> 10uF/4V
- Q14, Q17: value TSM9938HEUK+T -> MAX9938HEUK
- Q5: value FDC6324L -> FDC6330L
- R1: value 47R -> 300R
- R31, R32: value 1M -> 10K
- U2: value HRXL-MAXSONAR-WRC-MB7387 -> LE33; device elocktech_lib:HRXL-MAXSONAR-WRC-MB7387 -> elock_lib:LE33
Connections:
- removed net N$12: D7.A, R27.1
- removed net N$15: D8.A, R28.1
- removed net N$27: IC20.PGATE, Q22.G
- removed net N$29: IC20.ITH, R191.2
- removed net N$30: C162.1, R191.1
- removed net N$31: C161.1, IC20.RUN/SS, TP68.TP
- removed net N$33: D29.K, L13.1, Q22.D
- removed net N$37: C151.2, IC20.SENSE, Q22.S, R188.1
- removed net N$38: C159.1, IC20.VFB, R192.2, R196.1
- removed net N$53: Q17.VIN+, Q18-P.D, Q18-P.D1, R168.1
- removed net OUT_S3: D5.K, D7.K, J15.2, J16.2, Q8.D
- removed net OUT_S4: D6.K, D8.K, J15.3, J16.3, Q9.D
- new net N$41: JP1.1, JP2.1, R39.2
- new net N$42: J45.2, R46.2
- new net N$47: J45.3, R45.2
- new net N$48: C149.1, C150.1, C46.1, R47.1, R48.1, U2.VIN
- new net N$5: JP3.1, JP4.1, R38.2
- new net SMB-MEAS: Q17.VIN-, Q18-P.S, R168.2, R170.1
- net +3.3V: now also C45.1, U2.VOUT; no longer C159.2, L13.2, R192.1
- net +3.3V/2: now also J30.VCC; no longer U2.VCC
- net +5V: now also R47.2
- net +SMB: now also Q17.VIN+, R168.1, R48.2; no longer C149.1, C150.1, C151.1, IC20.MODE, IC20.VIN, Q18-P.S, R170.1, R188.2
- net 18V_GND: now also C39.2, C40.1, R39.1; no longer CN1.GND, JP2.1
- net 18V_SENSE: now also JP1.2; no longer CN1.PWR
- net ACT_S3_B: no longer Q9.G, R30.1
- net ACT_S4_B: no longer Q8.G, R29.1
- net B12_FEED: now also R42.2, R43.2; no longer R153.2, R155.2
- net BAT_GND: now also C41.2, C42.1, R38.1; no longer JP3.1, JP4.1
- net DCDC12VIN: now also R40.2, R41.2, R42.1, R43.1; no longer R153.1, R155.1
- net DGND: now also C3.2, C38.1, C40.2, C42.2, C43.-, C44.-, C45.2, C46.2, J30.GND, U2.INHIBIT; no longer C161.2, C162.2, C36.2, D25.A, D26.A, D29.A, D5.A, D6.A, D9.A, IC20.GND, J15.1, J16.1, Q8.S, Q9.S, R196.2, R29.2, R30.2
- net N$1: now also C38.2
- net N$19: now also C39.1
- net N$21: now also C41.1
- net N$4: now also R40.1, R41.1
- net N$49: now also C3.1
- net N$9: now also J30.EN; no longer U2.EN
- net OUT_S1: now also D25.A; no longer D25.K
- net OUT_S2: now also D26.A; no longer D26.K
- net P12V: now also C44.+
- net SMB_SCL: now also R46.1; no longer J45.2
- net SMB_SDA: now also R45.1; no longer J45.3
- net STR_FEED: now also R44.2; no longer R169.2
- net US-S_O: now also J30.SERIAL; no longer U2.SERIAL
- net VACT: now also C43.+, D25.K, D26.K; no longer C36.1, D9.C, J15.4, J16.4, R27.2, R28.2
- net VSUPLYACT: now also Q18-P.D, Q18-P.D1, R44.1; no longer Q17.VIN-, R168.2, R169.1
Other:
- note removed: "Vout= 1.23*(1+1.64/1M)"
- note removed: "Vout= 3.25V"
- moved on the sheet: C10, C134, C149, C150, C157, C7, D25, D26, D27, D31-1, D31-2, IC19P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
