File: PCB_KioskMB_r3.3-03.brd (EAGLE design)
At the start: 172.1 x 103.3 mm, 328 parts, among them IC1 ISL60002DIH325Z-TK, IC18 FT232RL, IC19 MCP6022-I/ST, IC2 SN65HVD12D, IC21 LTC1771EMS8, IC3 PIC24FJ256GA110-I/PT, IC4 PIC10F200T-I/OT, IC5 LM75ADP, IC6 24LC32A-I/MS, IC7 PCF2123TS/1-T, IC8 M25P16-VMN6P, IC9 LM3405AXMK/NOPB, J1 DF11-10DP-2DSA(01), J10 CCM03-3504LFT-NR, J14 3-641215-2, J15 1990834, J16 1990737, J17 14011213102000, J18 14011213102000, J19 14011213102000, J3 14011213102000, J30 22-11-2072, J4 3-641215-2, J45 3-641215-4, J47 DF11-10DP-2DSA(01), J48 3-641215-2, J49 3-641215-2, J50 0039301040, J7 SS-6566-NF, J8 TSW-108-07-G-D, J9 SS-6566-NF, Q14 MAX9938HEUK, Q15 SI4564DY, Q16 CSD87331Q3D, Q18 SI4564DY, Q19 CSD87331Q3D, Q2 FDC6330L, Q20 IPD30N06S2L-23, Q21 IPD30N06S2L-23, Q23 FDN352AP, Q24 BSS138, Q3 SR3.3.TCT, Q4 7B-28.63636MAAJ-T, Q5 FDC6330L, Q6 CM519 32.768KDZF-UT, Q7 SSM6P49NU,LFPZ, U1 LTC1955, U2 LE33, U3 ADS1015, U6 TPS43061, U7 TPS43061, U8 TPA3111D1PWP, U9 OPA322SAIDBVT, X1 FH12-10S-0.5S1.00MM, X2 MINI-USB_4P-85-32004-10X

Commit message: finalized bottom silk
finalized bottom silk, added 8 different revisions of bottom silk. added icons to match solar charger controller
Routing:
- net ID1_L_N: track 179.7 -> 183.0 mm
- net ID_L_P: track 186.1 -> 188.0 mm
Other:
- board text added: "10"
- board text added: "2"
- board text added: "3"
- board text added: "4"
- board text added: "5"
- board text added: "6"
- board text added: "7"
- board text added: "8"
- board text added: "9"
- board text added: "BAT+"
- board text added: "BAT-"
- board text added: "BTN 1"
- board text added: "BTN 2"
- board text added: "CELL MODEM"
- board text added: "CHG_CON_BAT+"
- board text added: "CHG_CON_BAT-"
- board text added: "CHG_CON_LOAD +"
- board text added: "CHG_CON_LOAD -"
- board text added: "CHG_CON_SOLAR+"
- board text added: "CHG_CON_SOLAR-"
- board text added: "CONNECT TO SOLAR PANEL"
- board text added: "CONTACT READER"
- board text added: "CONTACTLESS READER"
- board text added: "DOOR1"
- board text added: "DOOR2"
- board text added: "DOOR3"
- board text added: "DOOR4"
- board text added: "EXTRA POWER"
- board text added: "LED"
- board text added: "LIGHT+"
- board text added: "LIGHT-"
- board text added: "MIC+"
- board text added: "MIC-"
- board text added: "SENSORS"
- board text added: "SOLAR+IN"
- board text added: "SOLAR-IN"
- board text added: "STRIKE 1"
- board text added: "STRIKE 2"
- board text added: "STRIKE1"
- board text added: "STRIKE2"
- board text added: "ULTRA SONIC"
- board text added: "UPS+"
- board text added: "UPS-"
- board text removed: "BAT+SENSE IN"
- board text removed: "BAT+SENSE OUT"
- board text removed: "BAT-SENSE IN"
- board text removed: "BAT-SENSE OUT"
- board text removed: "DOOR 1"
- board text removed: "DOOR 2"
- board text removed: "HOPT SCHULER"
- board text removed: "ID_L+"
- board text removed: "ID_L-"
- board text removed: "MICROPHONE"
- board text removed: "V+SENSE IN"
- board text removed: "V+SENSE OUT"
- board text removed: "V-SENSE IN"
- board text removed: "V-SENSE OUT"
- board text removed: "VIN+"
